File: docs/kicad/ledBoard/ledBoard.sch (KiCad schematic (older format))
At the start: 13 parts

Commit message: docs - update/add more text labels for buttons and leds to schematics
Parts:
- J?: value Conn_01x08 -> LED_BOARD
Other:
- note added: "(REBOOT PI) PI_RUN"
- note added: "Bottom Button"
- note added: "I2S_RX_LED"
- note added: "I2S_TX_LED"
- note added: "In the Looper2 box,\nthe LEDS are in \nreverse order from \ntop to bottom"
- note added: "LED_PI_READY"
- note added: "LED_PI_RUN"
- note added: "ONBOARD_LED"
- note added: "TEENSY_PROG"
- note added: "Top Button"

Commit message: added breadboard for teensyPiLooper testing for new teensyExpression3
Parts:
- R?: value 220 -> 560
Changed lines of the file:
@@
 P 4550 3300
 F 0 "R?" V 4550 3600 50  0000 C CNN
-F 1 "220" V 4550 3300 50  0000 C CNN
+F 1 "560" V 4550 3300 50  0000 C CNN
 F 2 "" V 4480 3300 50  0001 C CNN
 F 3 "~" H 4550 3300 50  0001 C CNN
